Commit message: Добавлен correct_source.sh в корне воркспейса (microros_ros2_control) для корректного отображения обоих пакетов

File: src/microros_ros2_control_demos/urdf/test_cart_ft_sensor.xacro.urdf (robot description, URDF)
Before this commit: robot cartopole, 3 links, 2 joints
Links:
- link cart: geometry collision box size=0.5 0.5 0.2; visual box size=0.5 0.5 0.2
- link slideBar: geometry collision box size=30 0.05 0.05; visual box size=30 0.05 0.05

File: src/microros_ros2_control_demos/urdf/test_cart_position.xacro.urdf (robot description, URDF)
Before this commit: robot cartopole, 3 links, 2 joints
Links:
- link cart: geometry visual box size=0.5 0.5 0.2
- link slideBar: geometry visual box size=30 0.05 0.05
